Commit message: V1 Pool World

File: jelly_description/jelly_urdf/pool.urdf (robot description, URDF)
Before this commit: robot goal, 2 links, 1 joints
Links:
- removed link goal_base_link
- added link pool_base_link, mass 0.5; collision mesh ; visual mesh 
Joints:
- joint world_joint: child goal_base_link -> pool_base_link
